File: projects/pcb/udisk/ESP32-PICO-D4.sch (KiCad schematic (older format))
At the start: 3 parts

Commit message: feature(pcb): pcb ok
Parts:
- added AE1: ANT, ANT:AN9520, symbol Device:Antenna_Chip
- added C5: 0.1uF, Capacitor_SMD:C_0402_1005Metric, symbol Device:C_Small
- added C6, C7: NC, Capacitor_SMD:C_0402_1005Metric, symbol Device:C_Small
- added L1: NC, Inductor_SMD:L_0402_1005Metric, symbol Device:L_Small
- added R6: 10K, Resistor_SMD:R_0402_1005Metric, symbol Device:R
- C4: renamed from C?; footprint (none) -> Capacitor_SMD:C_0402_1005Metric
- R5: renamed from R?; footprint (none) -> Resistor_SMD:R_0402_1005Metric
- gave numbers to parts that had none: 1
Connections:
- net +3V3: now also R6.1
- net GND: now also C5.2, C6.2, C7.2
- net GPI34: now reaches U3.10 (IO34)
- net GPI35: now reaches U3.11 (IO35)
- net GPIO32: now reaches U3.12 (IO32)
- net GPIO33: now reaches U3.13 (IO33)
- net GPIO25: now reaches U3.14 (IO25)
- net GPIO26: now reaches U3.15 (IO26)
- net GPIO27: now reaches U3.16 (IO27)
- net GPIO14: now reaches U3.17 (IO14)
- net GPIO12: now reaches U3.18 (IO12)
- net at U3.2 (LNA_IN): now also C7.1, L1.1
- net GPIO13: now reaches U3.20 (IO13)
- net GPIO15: now reaches U3.21 (IO15)
- net GPIO2: now reaches U3.22 (IO2)
- net GPIO0: now reaches U3.23 (IO0)
- net GPIO0: now also R6.2
- net GPIO4: now reaches U3.24 (IO4)
- net GPIO5: now reaches U3.34 (IO5)
- net GPIO18: now reaches U3.35 (IO18)
- net GPIO23: now reaches U3.36 (IO23)
- net GPIO19: now reaches U3.38 (IO19)
- net GPIO22: now reaches U3.39 (IO22)
- net RXD: now reaches U3.40 (U0RXD/IO3)
- net TXD: now reaches U3.41 (U0TXD/IO1)
- net GPIO21: now reaches U3.42 (IO21)
- net GPI36: now reaches U3.5 (SENSOR_VP)
- net GPI39: now reaches U3.8 (SENSOR_VN)
- net EN: now reaches R5.2, U3.9 (EN)
- net EN: now also C5.1
- new net: AE1.1 (FEED), C6.1, L1.2
- no-connect marks 8 -> 13
Other:
- note added: "ESP32 has 6 strapping pins:\n• MTDI/GPIO12: internal pull-down\n• GPIO0: internal pull-up\n• GPIO2: internal pull-down\n• GPIO4: internal pull-down\n• MTDO/GPIO15: internal pull-up\n• GPIO5: internal pull-up"
- moved on the sheet: C4, R5
