File: projects/pcb/udisk/LCD160x80.sch (KiCad schematic (older format))
At the start: 6 parts, among them Q2 S8050

Commit message: feature(pcb): pcb ok
Parts:
- gave numbers to parts that had none: 1
Changed lines of the file:
@@
 $Descr A4 11693 8268
 encoding utf-8
-Sheet 3 4
+Sheet 3 5
 Title ""
 Date ""
@@
 AR Path="/5D355605" Ref="#PWR?"  Part="1"
 AR Path="/5D8B73CB/5D355605" Ref="#PWR019"  Part="1"
-F 0 "#PWR019" H 5150 3300 50  0001 C CNN
+AR Path="/5EE439BB/5D355605" Ref="#PWR0106"  Part="1"
+F 0 "#PWR0106" H 5150 3300 50  0001 C CNN
 F 1 "+3V3" H 5165 3623 50  0000 C CNN
 F 2 "" H 5150 3450 50  0001 C CNN
@@
 AR Path="/5D31AE1A/5D355606" Ref="C3"  Part="1"
 AR Path="/5D8B73CB/5D355606" Ref="C7"  Part="1"
-F 0 "C7" V 5198 3550 50  0000 C CNN
+AR Path="/5EE439BB/5D355606" Ref="C3"  Part="1"
+F 0 "C3" V 5198 3550 50  0000 C CNN
 F 1 "0.1uF" V 5289 3550 50  0000 C CNN
 F 2 "Capacitor_SMD:C_0402_1005Metric" H 5488 3400 50  0001 C CNN
@@
 AR Path="/5D355607" Ref="#PWR?"  Part="1"
 AR Path="/5D8B73CB/5D355607" Ref="#PWR020"  Part="1"
-F 0 "#PWR020" H 5600 3600 50  0001 C CNN
+AR Path="/5EE439BB/5D355607" Ref="#PWR0107"  Part="1"
+F 0 "#PWR0107" H 5600 3600 50  0001 C CNN
 F 1 "GND" H 5605 3677 50  0000 C CNN
 F 2 "" H 5600 3850 50  0001 C CNN
@@
 AR Path="/5D355608" Ref="#PWR?"  Part="1"
 AR Path="/5D8B73CB/5D355608" Ref="#PWR018"  Part="1"
-F 0 "#PWR018" H 4800 3800 50  0001 C CNN
+AR Path="/5EE439BB/5D355608" Ref="#PWR0108"  Part="1"
+F 0 "#PWR0108" H 4800 3800 50  0001 C CNN
 F 1 "GND" H 4805 3877 50  0000 C CNN
 F 2 "" H 4800 4050 50  0001 C CNN
@@
 AR Path="/5D31AE1A/5D355609" Ref="Q2"  Part="1"
 AR Path="/5D8B73CB/5D355609" Ref="Q3"  Part="1"
-F 0 "Q3" H 7041 3496 50  0000 L CNN
+AR Path="/5EE439BB/5D355609" Ref="Q1"  Part="1"
+F 0 "Q1" H 7041 3496 50  0000 L CNN
 F 1 "S8050" H 7041 3405 50  0000 L CNN
 F 2 "Package_TO_SOT_SMD:SOT-23" H 7050 3550 50  0001 C CNN
@@
 AR Path="/5D31AE1A/5D35560A" Ref="R9"  Part="1"
 AR Path="/5D8B73CB/5D35560A" Ref="R8"  Part="1"
-F 0 "R8" H 7020 2996 50  0000 L CNN
+AR Path="/5EE439BB/5D35560A" Ref="R4"  Part="1"
+F 0 "R4" H 7020 2996 50  0000 L CNN
 F 1 "10" H 7020 2905 50  0000 L CNN
 F 2 "Resistor_SMD:R_0402_1005Metric" V 6880 2950 50  0001 C CNN
@@
 AR Path="/5D35560B" Ref="#PWR?"  Part="1"
 AR Path="/5D8B73CB/5D35560B" Ref="#PWR022"  Part="1"
-F 0 "#PWR022" H 6950 3800 50  0001 C CNN
+AR Path="/5EE439BB/5D35560B" Ref="#PWR0109"  Part="1"
+F 0 "#PWR0109" H 6950 3800 50  0001 C CNN
 F 1 "GND" H 6955 3877 50  0000 C CNN
 F 2 "" H 6950 4050 50  0001 C CNN
@@
 AR Path="/5D31AE1A/5D35560C" Ref="R7"  Part="1"
 AR Path="/5D8B73CB/5D35560C" Ref="R6"  Part="1"
-F 0 "R6" V 6143 3450 50  0000 C CNN
+AR Path="/5EE439BB/5D35560C" Ref="R2"  Part="1"
+F 0 "R2" V 6143 3450 50  0000 C CNN
 F 1 "1K" V 6234 3450 50  0000 C CNN
 F 2 "Resistor_SMD:R_0402_1005Metric" V 6280 3450 50  0001 C CNN
@@
 AR Path="/5D31AE1A/5D31194C" Ref="R8"  Part="1"
 AR Path="/5D8B73CB/5D31194C" Ref="R7"  Part="1"
-F 0 "R7" H 6670 2996 50  0000 L CNN
+AR Path="/5EE439BB/5D31194C" Ref="R3"  Part="1"
+F 0 "R3" H 6670 2996 50  0000 L CNN
 F 1 "10K" H 6670 2905 50  0000 L CNN
 F 2 "Resistor_SMD:R_0402_1005Metric" V 6530 2950 50  0001 C CNN
@@
 AR Path="/5D312D22" Ref="#PWR?"  Part="1"
 AR Path="/5D8B73CB/5D312D22" Ref="#PWR021"  Part="1"
-F 0 "#PWR021" H 6600 2350 50  0001 C CNN
+AR Path="/5EE439BB/5D312D22" Ref="#PWR0110"  Part="1"
+F 0 "#PWR0110" H 6600 2350 50  0001 C CNN
 F 1 "+3V3" H 6615 2673 50  0000 C CNN
 F 2 "" H 6600 2500 50  0001 C CNN
@@
 	5550 3550 5600 3550
 $Comp
-L LCD:IPS0.9'160x80 LCD?
+L LCD:IPS0.9'160x80 LCD1
 U 1 1 5D8CB560
 P 4250 2600
-F 0 "LCD?" H 4283 2775 50  0000 C CNN
+F 0 "LCD1" H 4283 2775 50  0000 C CNN
 F 1 "IPS0.9'160x80" H 4283 2684 50  0000 C CNN
 F 2 "LCD:IPS0.9'160x80" H 4200 1200 50  0001 C CNN
