File: projects/pcb/udisk/POWER.sch (KiCad schematic (older format))
At the start: 4 parts

Commit message: feature(pcb): pcb ok
Parts:
- removed R?: 100K, Resistor_SMD:R_0402_1005Metric, symbol Device:R
- removed U?: RT9013, Package_TO_SOT_SMD:SOT-23-5, symbol LDO:RT9013
- added R1: 100K, Resistor_SMD:R_0402_1005Metric, symbol Device:R
- added U1: RT9013, Package_TO_SOT_SMD:SOT-23-5, symbol LDO:RT9013
- gave numbers to parts that had none: 2
Connections:
- net +3V3: now also U1.5 (OUT)
- net GND: now also U1.2 (GND)
- net +BATT renamed VBUS
- net VBUS: now also R1.2, U1.1 (IN)
- new net: R1.1, U1.3 (EN)
Changed lines of the file:
@@
 $Descr A4 11693 8268
 encoding utf-8
-Sheet 2 4
+Sheet 2 5
 Title ""
 Date ""
@@
 $EndDescr
 $Comp
-L LDO:RT9013 U?
-U 1 1 5D8B8399
+L LDO:RT9013 U1
+U 1 1 5EE439C6
 P 5900 3400
-F 0 "U?" H 5900 3765 50  0000 C CNN
+F 0 "U1" H 5900 3765 50  0000 C CNN
 F 1 "RT9013" H 5900 3674 50  0000 C CNN
 F 2 "Package_TO_SOT_SMD:SOT-23-5" H 6600 3100 50  0001 C CNN
@@
 $EndComp
 $Comp
-L Device:R R?
-U 1 1 5D8B87FE
+L Device:R R1
+U 1 1 5EE439C7
 P 5350 3400
-F 0 "R?" V 5143 3400 50  0000 C CNN
+F 0 "R1" V 5143 3400 50  0000 C CNN
 F 1 "100K" V 5234 3400 50  0000 C CNN
 F 2 "Resistor_SMD:R_0402_1005Metric" V 5280 3400 50  0001 C CNN
@@
 Wire Wire Line
 	5500 3400 5600 3400
-$Comp
-L power:+BATT #PWR?
-U 1 1 5D8B90D2
-P 5000 3000
-F 0 "#PWR?" H 5000 2850 50  0001 C CNN
-F 1 "+BATT" H 5015 3173 50  0000 C CNN
-F 2 "" H 5000 3000 50  0001 C CNN
-F 3 "" H 5000 3000 50  0001 C CNN
-	1    5000 3000
-	1    0    0    -1
-$EndComp
 Wire Wire Line
 	5000 3000 5000 3300
@@
 	5200 3300 5600 3300
 $Comp
-L power:GND #PWR?
+L power:GND #PWR0102
 U 1 1 5D8B98A8
 P 5900 4000
-F 0 "#PWR?" H 5900 3750 50  0001 C CNN
+F 0 "#PWR0102" H 5900 3750 50  0001 C CNN
 F 1 "GND" H 5905 3827 50  0000 C CNN
 F 2 "" H 5900 4000 50  0001 C CNN
@@
 	5900 3700 5900 4000
 $Comp
-L Device:C_Small C?
+L Device:C_Small C1
 U 1 1 5D8B9DEE
 P 5000 3550
-F 0 "C?" H 5092 3596 50  0000 L CNN
+F 0 "C1" H 5092 3596 50  0000 L CNN
 F 1 "1uF" H 5092 3505 50  0000 L CNN
 F 2 "Capacitor_SMD:C_0603_1608Metric" H 5000 3550 50  0001 C CNN
@@
 Connection ~ 5000 3300
 $Comp
-L power:GND #PWR?
-U 1 1 5D8BA916
+L power:GND #PWR0103
+U 1 1 5EE439CB
 P 5000 4000
-F 0 "#PWR?" H 5000 3750 50  0001 C CNN
+F 0 "#PWR0103" H 5000 3750 50  0001 C CNN
 F 1 "GND" H 5005 3827 50  0000 C CNN
 F 2 "" H 5000 4000 50  0001 C CNN
@@
 NoConn ~ 6200 3400
 $Comp
-L Device:C_Small C?
+L Device:C_Small C2
 U 1 1 5D8BB265
 P 6700 3550
-F 0 "C?" H 6792 3596 50  0000 L CNN
+F 0 "C2" H 6792 3596 50  0000 L CNN
 F 1 "1uF" H 6792 3505 50  0000 L CNN
 F 2 "Capacitor_SMD:C_0603_1608Metric" H 6700 3550 50  0001 C CNN
@@
 Connection ~ 6700 3300
 $Comp
-L power:GND #PWR?
+L power:GND #PWR0104
 U 1 1 5D8BBA4B
 P 6700 4000
-F 0 "#PWR?" H 6700 3750 50  0001 C CNN
+F 0 "#PWR0104" H 6700 3750 50  0001 C CNN
 F 1 "GND" H 6705 3827 50  0000 C CNN
 F 2 "" H 6700 4000 50  0001 C CNN
@@
 	6700 3650 6700 4000
 $Comp
-L power:+3V3 #PWR?
+L power:+3V3 #PWR0105
 U 1 1 5D8BC921
 P 6700 3000
-F 0 "#PWR?" H 6700 2850 50  0001 C CNN
+F 0 "#PWR0105" H 6700 2850 50  0001 C CNN
 F 1 "+3V3" H 6715 3173 50  0000 C CNN
 F 2 "" H 6700 3000 50  0001 C CNN
@@
 	1    0    0    -1
 $EndComp
+$Comp
+L power:VBUS #PWR0122
+U 1 1 5ED918E9
+P 5000 3000
+F 0 "#PWR0122" H 5000 2850 50  0001 C CNN
+F 1 "VBUS" H 5015 3173 50  0000 C CNN
+F 2 "" H 5000 3000 50  0001 C CNN
+F 3 "" H 5000 3000 50  0001 C CNN
+	1    5000 3000
+	1    0    0    -1
+$EndComp
