File: projects/pcb/udisk/udisk.kicad_pcb (KiCad board)
At the start: 2 copper layers, 13.6 x 50 mm, 27 parts, among them Q1 S8050, U1 RT9013, U2 APDS-9960, U3 ESP32-PICO-D4, U4 upcb, U5 udisk

Commit message: udisk ok
Parts:
- removed U4: upcb, USB:upcb
- added C8: 0.1uF, Capacitor_SMD:C_0402_1005Metric, F.Cu at (133.9, 51.3)
- added D1: WS2812B-0807, RGB_LED:WS2812B-0807, F.Cu at (133.9, 49.1)
- added G***: LOGO, udisk:love, B.Cu at (138.7, 33.9)
- added G***: LOGO, udisk:love, B.Cu at (129.2, 33.9)
- added J1: USB_A, USB:USB_A_2.0_Male, B.Cu at (133.9, 81.7)
- added REF**: OSHW-Symbol_6.7x6mm_SilkScreen, Symbol:OSHW-Symbol_6.7x6mm_SilkScreen, F.Cu at (133.9, 60.7)
- added TP5: GND, TestPoint:TestPoint_Pad_D1.0mm, F.Cu at (133.9, 76.2)
- moved C3 1.20 mm to (133.9, 52.4)
Connections:
- AE1 pad 2: Net-(AE1-Pad2) -> (no net)
- LCD1 pad 1: Net-(LCD1-Pad1) -> (no net)
- LCD1 pad 2: Net-(LCD1-Pad2) -> (no net)
- LCD1 pad 9: Net-(LCD1-Pad9) -> (no net)
- U1 pad 4: Net-(U1-Pad4) -> (no net)
- U2 pad 2: /APDS-9960/INT -> (no net)
- U3 pad 10: /ESP32-PICO-D4/GPI34 -> (no net)
- U3 pad 11: /ESP32-PICO-D4/GPI35 -> (no net)
- U3 pad 12: /ESP32-PICO-D4/GPIO32 -> (no net)
- U3 pad 13: /ESP32-PICO-D4/GPIO33 -> (no net)
- U3 pad 14: /ESP32-PICO-D4/GPIO25 -> (no net)
- U3 pad 15: /ESP32-PICO-D4/GPIO26 -> (no net)
- U3 pad 16: /ESP32-PICO-D4/GPIO27 -> (no net)
- U3 pad 18: /ESP32-PICO-D4/GPIO12 -> (no net)
- U3 pad 22: /ESP32-PICO-D4/GPIO2 -> (no net)
- U3 pad 24: /ESP32-PICO-D4/GPIO4 -> /DIN
- U3 pad 25: Net-(U3-Pad25) -> (no net)
- U3 pad 26: Net-(U3-Pad26) -> (no net)
- U3 pad 27: Net-(U3-Pad27) -> (no net)
- U3 pad 28: Net-(U3-Pad28) -> (no net)
- U3 pad 29: Net-(U3-Pad29) -> (no net)
- U3 pad 30: Net-(U3-Pad30) -> (no net)
- U3 pad 31: Net-(U3-Pad31) -> (no net)
- U3 pad 32: Net-(U3-Pad32) -> (no net)
- U3 pad 33: Net-(U3-Pad33) -> (no net)
- U3 pad 34: /ESP32-PICO-D4/GPIO5 -> (no net)
- U3 pad 44: Net-(U3-Pad44) -> (no net)
- U3 pad 45: Net-(U3-Pad45) -> (no net)
- U3 pad 47: Net-(U3-Pad47) -> (no net)
- U3 pad 48: Net-(U3-Pad48) -> (no net)
- U3 pad 5: /ESP32-PICO-D4/GPI36 -> (no net)
- U3 pad 6: Net-(U3-Pad6) -> (no net)
- U3 pad 7: Net-(U3-Pad7) -> (no net)
- U3 pad 8: /ESP32-PICO-D4/GPI39 -> (no net)
- U5 pad 5: Net-(U5-Pad5) -> (no net)
- U5 pad 6: Net-(U5-Pad6) -> (no net)
Routing:
- net GND: track 23.4 -> 13.6 mm, vias 24 -> 23
- net /DIN: track 0.00 -> 6.85 mm
- net VBUS: track 33.7 -> 30.9 mm
- net /D-: track 12.3 -> 9.45 mm
- net /D+: track 12.3 -> 9.45 mm
- net +3V3: track 83.1 -> 84.3 mm
- net /LCD_MOSI: track 14.3 -> 15.1 mm
- net (no net): vias 1 -> 0
Other:
- board size 13.6 x 50 mm -> 13.6 x 44.7 mm
- board text added: "JLCJLCJLCJLC"
- board text added: "XWX"
- board text added: "love memory © X Y"
- board text removed: "XWX&XY"
