File: projects/pcb/udisk/udisk.sch (KiCad schematic (older format))
At the start: 0 parts

Commit message: feature(pcb): pcb ok
Parts:
- added TP1: TXD, TestPoint:TestPoint_Pad_D1.0mm, symbol Connector:TestPoint
- added TP2: RXD, TestPoint:TestPoint_Pad_D1.0mm, symbol Connector:TestPoint
- added TP3: EN, TestPoint:TestPoint_Pad_D1.0mm, symbol Connector:TestPoint
- added TP4: GPIO0, TestPoint:TestPoint_Pad_D1.0mm, symbol Connector:TestPoint
- added U4: upcb, USB:upcb, symbol USB:upcb
- added U5: udisk, USB:udisk, symbol USB:udisk
Connections:
- new net D+: U4.3 (D+), U5.3 (D+)
- new net D-: U4.2 (D-), U5.2 (D-)
- new net ESP32-PICO-D4/EN: TP3.1
- new net ESP32-PICO-D4/GPIO0: TP4.1
- new net ESP32-PICO-D4/RXD: TP2.1
- new net ESP32-PICO-D4/TXD: TP1.1
- new net GND: U4.4 (GND), U5.4 (GND)
- new net VBUS: U4.1 (VCC), U5.1 (VCC)
- no-connect marks 0 -> 16

Commit message: udisk ok
Parts:
- removed U4: upcb, USB:upcb, symbol USB:upcb
- added C8: 0.1uF, Capacitor_SMD:C_0402_1005Metric, symbol Device:C_Small
- added D1: WS2812B-0807, RGB_LED:WS2812B-0807, symbol RGB_LED:WS2812B-0807
- added J1: USB_A, USB:USB_A_2.0_Male, symbol Connector:USB_A
- added TP5: GND, TestPoint:TestPoint_Pad_D1.0mm, symbol Connector:TestPoint
Connections:
- net labels added: +3V3, DIN
- wire segments 28 -> 43
Changed lines of the file:
@@
 	4000 3750 3450 3750
 NoConn ~ 6050 2800
-NoConn ~ 6050 2900
-NoConn ~ 6050 3000
 NoConn ~ 6050 3100
 NoConn ~ 6050 4300
@@
 $EndComp
 $Comp
-L USB:upcb U4
-U 1 1 5ED8FA78
-P 2700 2400
-F 0 "U4" V 3265 2092 50  0000 C CNN
-F 1 "upcb" V 3174 2092 50  0000 C CNN
-F 2 "USB:upcb" H 2750 2450 50  0001 C CNN
-F 3 "" H 2750 2450 50  0001 C CNN
-	1    2700 2400
-	0    -1   -1   0
-$EndComp
-$Comp
 L power:VBUS #PWR0101
 U 1 1 5ED921D0
@@
 Wire Wire Line
 	3500 1800 3500 2050
-Wire Wire Line
-	3500 2050 3300 2050
 $Comp
 L power:GND #PWR0121
@@
 	3500 2050 3950 2050
 Connection ~ 3500 2050
-Wire Wire Line
-	3300 2150 3950 2150
 Wire Wire Line
 	3300 2250 3950 2250
@@
 	6050 3900 6500 3900
 NoConn ~ 6050 4200
+$Comp
+L Connector:USB_A J1
+U 1 1 5ED69406
+P 2650 2250
+F 0 "J1" H 2707 2717 50  0000 C CNN
+F 1 "USB_A" H 2707 2626 50  0000 C CNN
+F 2 "USB:USB_A_2.0_Male" H 2800 2200 50  0001 C CNN
+F 3 " ~" H 2800 2200 50  0001 C CNN
+	1    2650 2250
+	1    0    0    -1
+$EndComp
+Wire Wire Line
+	3300 2150 3950 2150
+Wire Wire Line
+	2950 2050 3500 2050
+Wire Wire Line
+	2650 2650 3300 2650
+Wire Wire Line
+	3300 2650 3300 2350
+Wire Wire Line
+	2950 2250 3150 2250
+Wire Wire Line
+	2950 2350 3150 2350
+Text Label 3150 2350 2    50   ~ 0
+D-
+Text Label 3150 2250 2    50   ~ 0
+D+
+Wire Wire Line
+	2650 2650 2550 2650
+Connection ~ 2650 2650
+Wire Wire Line
+	8250 4950 8250 5150
+$Comp
+L Device:C_Small C?
+U 1 1 5F28B88D
+P 8250 4850
+AR Path="/5ED81B08/5F28B88D" Ref="C?"  Part="1"
+AR Path="/5F28B88D" Ref="C8"  Part="1"
+F 0 "C8" H 8342 4896 50  0000 L CNN
+F 1 "0.1uF" H 8342 4805 50  0000 L CNN
+F 2 "Capacitor_SMD:C_0402_1005Metric" H 8250 4850 50  0001 C CNN
+F 3 "~" H 8250 4850 50  0001 C CNN
+	1    8250 4850
+	1    0    0    -1
+$EndComp
+Wire Wire Line
+	7600 5150 8250 5150
+Wire Wire Line
+	8250 4750 8250 4550
+Wire Wire Line
+	7600 4550 8250 4550
+$Comp
+L RGB_LED:WS2812B-0807 D?
+U 1 1 5F28B896
+P 7600 4850
+AR Path="/5ED81B08/5F28B896" Ref="D?"  Part="1"
+AR Path="/5F28B896" Ref="D1"  Part="1"
+F 0 "D1" H 7944 4896 50  0000 L CNN
+F 1 "WS2812B-0807" H 7944 4805 50  0000 L CNN
+F 2 "RGB_LED:WS2812B-0807" H 8150 4400 50  0001 C CNN
+F 3 "" H 7450 5100 50  0001 C CNN
+	1    7600 4850
+	1    0    0    -1
+$EndComp
+$Comp
+L power:+3V3 #PWR?
+U 1 1 5F29CBAD
+P 7600 4400
+AR Path="/5D8A8C31/5F29CBAD" Ref="#PWR?"  Part="1"
+AR Path="/5F29CBAD" Ref="#PWR0120"  Part="1"
+F 0 "#PWR0120" H 7600 4250 50  0001 C CNN
+F 1 "+3V3" H 7615 4573 50  0000 C CNN
+F 2 "" H 7600 4400 50  0001 C CNN
+F 3 "" H 7600 4400 50  0001 C CNN
+	1    7600 4400
+	1    0    0    -1
+$EndComp
+Wire Wire Line
+	7600 4400 7600 4550
+Connection ~ 7600 4550
+$Comp
+L power:GND #PWR0123
+U 1 1 5F29F0FB
+P 7600 5350
+F 0 "#PWR0123" H 7600 5100 50  0001 C CNN
+F 1 "GND" H 7605 5177 50  0000 C CNN
+F 2 "" H 7600 5350 50  0001 C CNN
+F 3 "" H 7600 5350 50  0001 C CNN
+	1    7600 5350
+	1    0    0    -1
+$EndComp
+Wire Wire Line
+	7600 5150 7600 5350
+Connection ~ 7600 5150
+NoConn ~ 7900 4850
+Wire Wire Line
+	7300 4850 7000 4850
+Wire Wire Line
+	6050 2900 6500 2900
+Text Label 6500 2900 2    50   ~ 0
+DIN
+Text Label 7000 4850 0    50   ~ 0
+DIN
+NoConn ~ 6050 3000
+$Comp
+L Connector:TestPoint TP5
+U 1 1 5EDCAAD1
+P 3450 3850
+F 0 "TP5" V 3450 4100 50  0000 C CNN
+F 1 "GND" V 3500 3750 50  0000 C CNN
+F 2 "TestPoint:TestPoint_Pad_D1.0mm" H 3650 3850 50  0001 C CNN
+F 3 "~" H 3650 3850 50  0001 C CNN
+	1    3450 3850
+	0    -1   -1   0
+$EndComp
+$Comp
+L power:GND #PWR0124
+U 1 1 5EDD0C6D
+P 3700 4050
+F 0 "#PWR0124" H 3700 3800 50  0001 C CNN
+F 1 "GND" H 3705 3877 50  0000 C CNN
+F 2 "" H 3700 4050 50  0001 C CNN
+F 3 "" H 3700 4050 50  0001 C CNN
+	1    3700 4050
+	1    0    0    -1
+$EndComp
+Wire Wire Line
+	3450 3850 3700 3850
+Wire Wire Line
+	3700 3850 3700 4050
 $EndSCHEMATC
